File: Board Design/Custom_Board_F303_Rev0.0/Custom_Board_F303_Rev0.0.kicad_sch (KiCad schematic)
At the start: 13 parts, among them U1 STM32F303RETx, X1 ABS25-32.768KHZ-6-T

Commit message: Added Schematic Components.
Parts:
- added C16, C17: 10p, symbol Device:C
- added J1: Conn_01x04_Pin, symbol Connector:Conn_01x04_Pin
- added Y1: 12MHz, symbol Device:Crystal_GND24
Connections:
- net +3.3V: now also J1.1 (Pin_1)
- net GND: now also C16.2, C17.2, J1.4 (Pin_4), Y1.2, Y1.4
- net SWCLK: now also J1.3 (Pin_3)
- net SWDIO: now also J1.2 (Pin_2)
- net I2C2_SCL: now reaches U1.42 (PA9)
- net I2C2_SDA: now reaches U1.43 (PA10)
- net HSE_IN: now reaches U1.5 (PF0)
- net HSE_IN: now also C16.1, Y1.1
- net I2C1_SCL: now reaches U1.50 (PA15)
- net I2C1_SDA: now reaches U1.59 (PB7)
- net HSE_OUT: now reaches U1.6 (PF1)
- net HSE_OUT: now also C17.1, Y1.3
- net LSE OSC_IN renamed LSE_IN
- net LSE OSC_OUT renamed LSE_OUT
Other:
- moved on the sheet: C1, C13, C14, C2, C3, C4, C5, C6, FB1, R2, U1, X1
